File: i2c_io_expander.brd (EAGLE design)
At the start: 55.5 x 51 mm, 21 parts, among them IC1 MCP23017SP, J1 43814-6621, J6 22-23-2031

Commit message: Added contact info and rev # to silkscreen Added VCC and GND designator to silkscreen
Parts:
- R1: value 120 -> 200
- R2: value 120 -> 110
- R3, R4: value 4k7 -> 2k7
Other:
- board text added: "GND"
- board text added: "VCC"
Changed lines of the file:
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@@
 <text x="11.8364" y="25.8826" size="1.016" layer="21">www.github.com/jes1510</text>
 <text x="11.557" y="23.8506" size="1.016" layer="21">12032015</text>
+<text x="54.229" y="21.9202" size="1.016" layer="21" rot="R90">VCC</text>
+<text x="54.0258" y="32.1056" size="1.016" layer="21" rot="R90">GND</text>
 </plain>
 <attributes>
@@
 <attribute name="MF" value="" x="3.7338" y="15.367" size="1.778" layer="27" display="off"/>
 </element>
-<element name="R1" library="rcl" package="R0603" value="120" x="3.8862" y="10.668" rot="R270">
+<element name="R1" library="rcl" package="R0603" value="200" x="3.8862" y="10.668" rot="R270">
 <attribute name="OC_NEWARK" value="unknown" x="3.8862" y="10.668" size="1.778" layer="27" rot="R270" display="off"/>
 <attribute name="MPN" value="" x="3.8862" y="10.668" size="1.778" layer="27" rot="R270" display="off"/>
 <attribute name="MF" value="" x="3.8862" y="10.668" size="1.778" layer="27" rot="R270" display="off"/>
 </element>
-<element name="R2" library="rcl" package="R0603" value="120" x="40.5638" y="21.717" rot="R270">
+<element name="R2" library="rcl" package="R0603" value="110" x="40.5638" y="21.717" rot="R270">
 <attribute name="OC_NEWARK" value="unknown" x="40.5638" y="21.717" size="1.778" layer="27" rot="R270" display="off"/>
 <attribute name="MPN" value="" x="40.5638" y="21.717" size="1.778" layer="27" rot="R270" display="off"/>
 <attribute name="MF" value="" x="40.5638" y="21.717" size="1.778" layer="27" rot="R270" display="off"/>
 </element>
-<element name="R3" library="rcl" package="R0603" value="4k7" x="41.8338" y="10.287" rot="R90">
+<element name="R3" library="rcl" package="R0603" value="2k7" x="41.8338" y="10.287" rot="R90">
 <attribute name="OC_NEWARK" value="unknown" x="41.8338" y="10.287" size="1.778" layer="27" rot="R90" display="off"/>
 <attribute name="MPN" value="" x="41.8338" y="10.287" size="1.778" layer="27" rot="R90" display="off"/>
 <attribute name="MF" value="" x="41.8338" y="10.287" size="1.778" layer="27" rot="R90" display="off"/>
 </element>
-<element name="R4" library="rcl" package="R0603" value="4k7" x="47.752" y="10.2362" rot="R90">
+<element name="R4" library="rcl" package="R0603" value="2k7" x="47.752" y="10.2362" rot="R90">
 <attribute name="OC_NEWARK" value="unknown" x="47.752" y="10.2362" size="1.778" layer="27" rot="R90" display="off"/>
 <attribute name="MPN" value="" x="47.752" y="10.2362" size="1.778" layer="27" rot="R90" display="off"/>
